File: hardware/esp32.kicad_pcb (KiCad board)
At the start: 4 copper layers, 60 x 40 mm, 79 parts, among them J101 USB-C-2, P101 PWR, P201 CON-SENSOR2, P202 CON-SENSOR2, P203 CON-SENSOR2, P204 CON-SENSOR2, P205 CON-SENSOR2, P206 CON-SENSOR2, Q101 NPN, Q102 NPN, U101 82400152, U102 AZ1117E-3.3V, U103 CP2102N-A02-GQFN24R, U104 ESP32-WROOM-32, U201 74AHC244, U202 74AHC244, U203 74AHC244

Commit message: routing finished
Parts:
- removed C2: TBD, kicad-libraries:R0402F
- removed R102: 1k, kicad-libraries:R0402F
- added D105: green, kicad-libraries:D0603F, F.Cu at (157.8, 125.5)
- added Fiducial_Mark: VAL**, kicad-libraries:Fiducial_Mark, F.Cu at (172.3, 146.2)
- added Fiducial_Mark: VAL**, kicad-libraries:Fiducial_Mark, F.Cu at (119.8, 157.2)
- added Fiducial_Mark: VAL**, kicad-libraries:Fiducial_Mark, F.Cu at (122.8, 125.7)
- added G***: LOGO, kicad-libraries:Logo_31x31, F.Cu at (135.7, 142.8)
- added RP104: 1k, kicad-libraries:4X0402, F.Cu at (146.0, 136.6)
- added RP105: 1k, kicad-libraries:4X0402, F.Cu at (157.1, 128.9)
- added VAL: WEEE_7mm, kicad-libraries:WEEE_7mm, B.Cu at (153.8, 143.7)
- added VAL: CE_5mm, kicad-libraries:CE_5mm, B.Cu at (133.8, 143.7)
- moved R3 122.7 mm to (120.4, 136.7), turned to 270 degrees
- moved R2 115.5 mm to (125.8, 130.3), turned to 180 degrees
- moved R4 110.1 mm to (120.4, 151.7), turned to 270 degrees
- moved R1 98.0 mm to (140.8, 130.2), turned to 180 degrees
- moved R202 91.6 mm to (141.8, 157.1)
- moved R201 87.5 mm to (126.8, 157.1)
- moved C202 86.3 mm to (129.2, 139.8)
- moved C203 78.9 mm to (131.9, 153.8), turned to 180 degrees
- moved C201 76.2 mm to (136.7, 133.6)
- moved RP206 7.32 mm to (144.8, 155.4)
- moved CP206 4.74 mm to (141.8, 155.4), turned to 90 degrees
- moved CP201 4.51 mm to (140.8, 131.8), turned to 270 degrees
- moved CP202 3.70 mm to (125.8, 131.8), turned to 270 degrees
- moved U203 2.53 mm to (134.3, 149.8), turned to 90 degrees
- moved U202 2.00 mm to (126.8, 143.7), turned to 270 degrees
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Connections:
- net Net-(C102-Pad1) renamed USB_GND
- net Net-(C102-Pad2) renamed USB_5V
- RP101 pad 1: B0-CLK -> B0-MISO
- RP101 pad 2: B0-MISO -> B0-CLK
- RP201 pad 1: Net-(CP201-Pad1) -> B0-CS0
- RP201 pad 2: Net-(CP201-Pad2) -> Net-(RP201-Pad2)
- RP201 pad 3: Net-(CP201-Pad3) -> Net-(RP201-Pad3)
- RP201 pad 4: Net-(P201-Pad7) -> Net-(RP201-Pad4)
- RP201 pad 5: Net-(RP201-Pad5) -> Net-(P201-Pad7)
- RP201 pad 6: Net-(RP201-Pad6) -> Net-(CP201-Pad3)
- RP201 pad 7: Net-(RP201-Pad7) -> Net-(CP201-Pad2)
- RP201 pad 8: B0-CS0 -> Net-(CP201-Pad1)
- RP202 pad 1: Net-(CP202-Pad1) -> B0-CS1
- RP202 pad 2: Net-(CP202-Pad2) -> Net-(RP202-Pad2)
- RP202 pad 3: Net-(CP202-Pad3) -> Net-(RP202-Pad3)
- RP202 pad 4: Net-(P202-Pad7) -> Net-(RP202-Pad4)
- RP202 pad 5: Net-(RP202-Pad5) -> Net-(P202-Pad7)
- RP202 pad 6: Net-(RP202-Pad6) -> Net-(CP202-Pad3)
- RP202 pad 7: Net-(RP202-Pad7) -> Net-(CP202-Pad2)
- RP202 pad 8: B0-CS1 -> Net-(CP202-Pad1)
- RP203 pad 1: Net-(CP203-Pad1) -> B0-CS2
- RP203 pad 2: Net-(CP203-Pad2) -> Net-(RP203-Pad2)
- RP203 pad 3: Net-(CP203-Pad3) -> Net-(RP203-Pad3)
- RP203 pad 4: Net-(P203-Pad7) -> Net-(RP203-Pad4)
- RP203 pad 5: Net-(RP203-Pad5) -> Net-(P203-Pad7)
- RP203 pad 6: Net-(RP203-Pad6) -> Net-(CP203-Pad3)
- RP203 pad 7: Net-(RP203-Pad7) -> Net-(CP203-Pad2)
- RP203 pad 8: B0-CS2 -> Net-(CP203-Pad1)
- RP204 pad 1: Net-(CP204-Pad1) -> B1-CS0
- RP204 pad 2: Net-(CP204-Pad2) -> Net-(RP204-Pad2)
- RP204 pad 3: Net-(CP204-Pad3) -> Net-(RP204-Pad3)
- RP204 pad 4: Net-(P204-Pad7) -> Net-(RP204-Pad4)
- RP204 pad 5: Net-(RP204-Pad5) -> Net-(P204-Pad7)
- RP204 pad 6: Net-(RP204-Pad6) -> Net-(CP204-Pad3)
- RP204 pad 7: Net-(RP204-Pad7) -> Net-(CP204-Pad2)
- RP204 pad 8: B1-CS0 -> Net-(CP204-Pad1)
- RP205 pad 1: Net-(CP205-Pad1) -> B1-CS1
- RP205 pad 2: Net-(CP205-Pad2) -> Net-(RP205-Pad2)
- RP205 pad 3: Net-(CP205-Pad3) -> Net-(RP205-Pad3)
- RP205 pad 4: Net-(P205-Pad7) -> Net-(RP205-Pad4)
- RP205 pad 5: Net-(RP205-Pad5) -> Net-(P205-Pad7)
- RP205 pad 6: Net-(RP205-Pad6) -> Net-(CP205-Pad3)
- RP205 pad 7: Net-(RP205-Pad7) -> Net-(CP205-Pad2)
- RP205 pad 8: B1-CS1 -> Net-(CP205-Pad1)
- RP206 pad 1: Net-(CP206-Pad1) -> B1-CS2
- RP206 pad 2: Net-(CP206-Pad2) -> Net-(RP206-Pad2)
- RP206 pad 3: Net-(CP206-Pad3) -> Net-(RP206-Pad3)
- RP206 pad 4: Net-(P206-Pad7) -> Net-(RP206-Pad4)
- RP206 pad 5: Net-(RP206-Pad5) -> Net-(P206-Pad7)
- RP206 pad 6: Net-(RP206-Pad6) -> Net-(CP206-Pad3)
- RP206 pad 7: Net-(RP206-Pad7) -> Net-(CP206-Pad2)
- RP206 pad 8: B1-CS2 -> Net-(CP206-Pad1)
- U104 pad 10: Net-(U104-Pad10) -> B0-CS2
- U104 pad 11: Net-(U104-Pad11) -> B0-CS1
- U104 pad 12: Net-(U104-Pad12) -> B0-CS0
- U104 pad 13: Net-(RP101-Pad8) -> Net-(RP101-Pad7)
- U104 pad 14: Net-(RP101-Pad7) -> Net-(RP101-Pad8)
- U104 pad 27: Net-(U104-Pad27) -> B1-CS2
- U104 pad 28: Net-(U104-Pad28) -> B1-CS0
- U104 pad 4: Net-(U104-Pad4) -> ESP_ADC_5V
- U104 pad 5: Net-(U104-Pad5) -> ESP_ADC_VUSB
- U104 pad 9: Net-(U104-Pad9) -> B1-CS1
- U201 pad 11: Net-(RP202-Pad5) -> Net-(RP202-Pad4)
- U201 pad 14: Net-(RP201-Pad6) -> Net-(RP201-Pad3)
- U201 pad 16: Net-(RP201-Pad7) -> Net-(RP201-Pad2)
- U201 pad 5: Net-(RP202-Pad7) -> Net-(RP202-Pad2)
- U201 pad 7: Net-(RP202-Pad6) -> Net-(RP202-Pad3)
- U201 pad 8: Net-(RP201-Pad5) -> Net-(RP201-Pad4)
- U202 pad 11: Net-(RP204-Pad5) -> Net-(RP204-Pad4)
- U202 pad 14: Net-(RP203-Pad6) -> Net-(RP203-Pad3)
- U202 pad 16: Net-(RP203-Pad7) -> Net-(RP203-Pad2)
- U202 pad 5: Net-(RP204-Pad7) -> Net-(RP204-Pad2)
- U202 pad 7: Net-(RP204-Pad6) -> Net-(RP204-Pad3)
- U202 pad 8: Net-(RP203-Pad5) -> Net-(RP203-Pad4)
- U203 pad 11: Net-(RP206-Pad5) -> Net-(RP206-Pad4)
- U203 pad 14: Net-(RP205-Pad6) -> Net-(RP205-Pad3)
- U203 pad 16: Net-(RP205-Pad7) -> Net-(RP205-Pad2)
- U203 pad 5: Net-(RP206-Pad7) -> Net-(RP206-Pad2)
- U203 pad 7: Net-(RP206-Pad6) -> Net-(RP206-Pad3)
- U203 pad 8: Net-(RP205-Pad5) -> Net-(RP205-Pad4)
Routing:
- net GND: track 2.36 -> 127.3 mm, vias 0 -> 132
- net B1-CS0: track 0.00 -> 64.6 mm, vias 0 -> 2
- net 3V3: track 0.00 -> 52.5 mm, vias 0 -> 42
- net B0-CS2: track 0.00 -> 48.5 mm, vias 0 -> 3
- net B1-CS1: track 0.00 -> 48.3 mm, vias 0 -> 2
- net B0-CS1: track 0.00 -> 46.2 mm, vias 0 -> 4
- net B1-CLK: track 0.00 -> 37.9 mm, vias 0 -> 2
- net B1-MISO: track 0.00 -> 36.2 mm, vias 0 -> 2
- net B1-CS2: track 0.00 -> 35.8 mm, vias 0 -> 3
- net B1-MOSI: track 0.00 -> 34.7 mm
- net B0-CS0: track 0.00 -> 33.6 mm, vias 0 -> 2
- net 5V: track 33.6 -> 65.3 mm, vias 0 -> 31
- net Net-(Q101-PadE): track 0.82 -> 31.5 mm, vias 1 -> 2
- net USB_5V: track 0.00 -> 29.6 mm, vias 0 -> 4
- net ESP_ADC_5V: track 0.00 -> 27.3 mm, vias 0 -> 2
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- added copper zone on F.Cu, net 3V3
- added copper zone on VCC, net 3V3
- added copper zone on F.Cu, net 5V
- added copper zone on VCC, net 5V
- added copper zone on F.Cu, net GND
- added copper zone on GND, net GND
- added copper zone on F.Cu, net USB_5V
- added copper zone on F.Cu, net USB_GND
Other:
- board text added: "0"
- board text added: "1"
- board text added: "ESP32 1.0"
- board text added: "tinkerforge.com"

Commit message: version 1.0 finished
Parts:
- moved Fiducial_Mark 1.12 mm to (120.8, 157.7)
Other:
- board text added: "A"
- board text added: "B"
- board text added: "C"
- board text added: "D"
- board text added: "E"
- board text added: "F"
